Commit message: laser scan sub node

File: k2wr_description/urdf/k2wr.xacro (robot description, xacro)
@@ -102,5 +102,5 @@
   </link>
   <joint name="camera_joint" type="fixed">
-    <origin xyz="0.2 0.0 0.0" rpy="0.0 0.0 0.0"/>
+    <origin xyz="0.25 0.0 0.0" rpy="0.0 0.0 0.0"/>
     <parent link="link_chassis"/>
     <child link="camera_link"/>
